File: reality-from-scratch-motherboard.kicad_sch (KiCad schematic)
At the start: 12 parts, among them IC1 ICM-42688-P, U1 RP2040

Commit message: schematics first revision done
Parts:
- removed C1, C2, C3, C4, C5, C6, C7: 100nF, symbol Device:C
- added C101: 1uF/10V, symbol Device:C
- added C102, C103: 100nF, Capacitor_SMD:C_0402_1005Metric, symbol Device:C
- added C104: 1uF, Capacitor_SMD:C_0402_1005Metric, symbol Device:C
- added C105: 100n, Capacitor_SMD:C_0402_1005Metric, symbol Device:C
- added C106, C107, C110: 10u, Capacitor_SMD:C_0805_2012Metric, symbol Device:C
- added C108, C109: 15p, Capacitor_SMD:C_0402_1005Metric, symbol Device:C
- added C111, C112, C113, C114, C115, C116, C117: 100nF, symbol Device:C
- added D101: LED, symbol Device:LED
- added H101, H102, H103, H104: MountingHole, MountingHole:MountingHole_2.7mm_M2.5, symbol Mechanical:MountingHole
- added J102: TC2050-IDC, Connector:Tag-Connect_TC2050-IDC-FP_2x05_P1.27mm_Vertical, symbol TC2050-IDC:TC2050-IDC
- added R101, R105: 1k, Resistor_SMD:R_0402_1005Metric, symbol Device:R
- added R102: 10kΩ/1%, Resistor_SMD:R_0402_1005Metric, symbol Device:R
- added R103, R104: 5.1K, Resistor_SMD:R_0402_1005Metric, symbol Device:R
- added R106, R107: 27Ω, symbol Device:R
- added R108: 1kΩ, symbol Device:R
- added TP101: Test_1V1, symbol Connector:TestPoint
- added TP102: Test_3V3, symbol Connector:TestPoint
- added U101: W25Q128JVS, Package_SO:SOIC-8_5.23x5.23mm_P1.27mm, symbol Memory_Flash:W25Q128JVS
- added U102: USB-TYPE-C-018, footprint:USB-C_SMD-TYPE-C-31-M-12, symbol USB-TYPE-C-018:USB-TYPE-C-018
- added U103: NCP1117-3.3_SOT223, Package_TO_SOT_SMD:SOT-223-3_TabPin2, symbol Regulator_Linear:NCP1117-3.3_SOT223
- added U104: TS-1187A-B-A-B, footprint:SW-SMD_4P-L5.1-W5.1-P3.70-LS6.5-TL-2, symbol TS-1187A-B-A-B:TS-1187A-B-A-B
- added X101: X322512MSB4SI, footprints:OSC-SMD_4P-L3.2-W2.5-BL, symbol X322512MSB4SI:X322512MSB4SI
- C10: value 2.2uF -> 2.2uF/10V
- C9: value 0.1uF -> 0.1uF/10V
Connections:
- net +3.3V: now also C101.1, C111.1, C112.1, C113.1, C114.1, C115.1, C116.1, C117.1, TP102.1
- net GND: now also IC1.10 (RESV_4), IC1.11 (RESV_5), IC1.2 (RESV_1), IC1.3 (RESV_2), IC1.6 (GND), IC1.7 (RESV_3), U1.19 (TESTEN), U1.57 (GND), C101.2, C102.2, C103.2, C104.2, C105.2, C106.2, C107.2, C108.2, C109.2, C110.2, C111.2, C112.2, C113.2, C114.2, C115.2, C116.2, C117.2, D101.1 (K), J102.4, R103.1, R104.2, U101.4 (GND), U102.0 (SH), U102.13 (SH), U102.2 (SH), U102.3 (SH), U102.A1 (GND), U102.A12 (GND), U102.B1 (GND), U102.B12 (GND), U103.1 (GND), U104.4 (D), X101.2 (GND), X101.4 (GND)
- net SDO: now reaches IC1.1 (AP_SDO_/_AP_AD0)
- net SDO: now also U1.2 (GPIO0)
- net CS: now reaches IC1.12 (AP_CS)
- net CS: now also U1.3 (GPIO1)
- net SCLK: now reaches IC1.13 (AP_SCL_/_AP_SCLK)
- net SCLK: now also U1.4 (GPIO2)
- net SDI: now reaches IC1.14 (AP_SDA_/_AP_SDIO_/_AP_SDI)
- net SDI: now also U1.5 (GPIO3)
- net INT1: now reaches IC1.4 (INT1_/_INT)
- net INT1: now also U1.7 (GPIO5)
- net INT2: now reaches IC1.9 (INT2_/_FSYNC_/_CLKIN)
- net INT2: now also U1.6 (GPIO4)
- net UART1_TX: now reaches U1.11 (GPIO8)
- net UART1_TX: now also J102.10
- net UART1_RX: now reaches U1.12 (GPIO9)
- net UART1_RX: now also J102.9
- net XIN: now reaches U1.20 (XIN)
- net XIN: now also C108.1, X101.3 (OSC2)
- net XOUT: now reaches U1.21 (XOUT)
- net XOUT: now also R105.1
- net +1V1: now reaches U1.23 (DVDD), U1.50 (DVDD)
- net +1V1: now also U1.45 (VREG_VOUT), C102.1, C103.1, C104.1, TP101.1
- net SWCLK: now reaches U1.24 (SWCLK)
- net SWCLK: now also J102.2
- net SWD: now reaches U1.25 (SWD)
- net SWD: now also J102.1
- net RUN: now reaches U1.26 (RUN)
- net RUN: now also J102.5
- net LED_HB: now reaches U1.37 (GPIO25)
- net LED_HB: now also R108.2
- net at U1.46 (USB_DM): now also R107.2
- net at U1.47 (USB_DP): now also R106.2
- net QSPI_SD3: now reaches U1.51 (QSPI_SD3)
- net QSPI_SD3: now also U101.7 (IO3)
- net QSPI_SCLK: now reaches U1.52 (QSPI_SCLK)
- net QSPI_SCLK: now also U101.6 (CLK)
- net QSPI_SD0: now reaches U1.53 (QSPI_SD0)
- net QSPI_SD0: now also U101.5 (DI(IO0))
- net QSPI_SD2: now reaches U1.54 (QSPI_SD2)
- net QSPI_SD2: now also U101.3 (IO2)
- net QSPI_SD1: now reaches U1.55 (QSPI_SD1)
- net QSPI_SD1: now also U101.2 (DO(IO1))
- net QSPI_SS: now reaches U1.56 (QSPI_SS)
- net QSPI_SS: now also R101.1, R102.2, U101.1 (~{CS})
- new net: D101.2 (A), R108.1
- new net: C109.1, R105.2, X101.1 (OSC1)
- new net: R104.1, U102.A5 (CC1)
- new net: R103.2, U102.B5 (CC2)
- new net: R101.2, U104.2 (B)
- new net +3V3: C105.1, C107.1, C110.1, J102.3, R102.1, U101.8 (VCC), U103.2 (VO)
- new net +5V: C106.1, U102.A4 (VBUS), U102.A9 (VBUS), U102.B4 (VBUS), U102.B9 (VBUS), U103.3 (VI)
- new net USB_N: R107.1, U102.A7 (DN1), U102.B7 (DN2)
- new net USB_P: R106.1, U102.A6 (DP1), U102.B6 (DP2)
- no-connect marks 0 -> 10
Other:
- note added: "Crystal"
- note added: "Flash"
- note added: "Make sure C101 is close to pin 44 of RP2040"
- note added: "Make sure C104 is close to pin 45 of RP2040"
- note added: "Place C8 close to VDDIO"
- moved on the sheet: C10, C8, C9, IC1, U1

Commit message: fixed MD file
Parts:
- removed H103, H104: MountingHole, MountingHole:MountingHole_2.7mm_M2.5, symbol Mechanical:MountingHole
- added TP103: Test_5V5, TestPoint:TestPoint_Pad_D1.5mm, symbol Connector:TestPoint
- C10, C101, C111, C112, C113, C114, C115, C116, C117, C8, C9, R106, R107, R108: footprint (none) -> Capacitor_SMD:C_0402_1005Metric
- C106, C107, C110: footprint Capacitor_SMD:C_0805_2012Metric -> Capacitor_SMD:C_0402_1005Metric
- C108, C109: value 15p -> 15pF
- D101: footprint (none) -> LED_SMD:LED_0603_1608Metric
- IC1: footprint IIM42352 -> footprints:IIM42352
- TP101, TP102: footprint (none) -> TestPoint:TestPoint_Pad_D1.5mm
- U102: footprint footprint:USB-C_SMD-TYPE-C-31-M-12 -> footprints:USB-C_SMD-TYPE-C-31-M-12
- U104: footprint footprint:SW-SMD_4P-L5.1-W5.1-P3.70-LS6.5-TL-2 -> footprints:SW-SMD_4P-L5.1-W5.1-P3.70-LS6.5-TL-2
Connections:
- net +3.3V is gone; now on net +3V3: C10.1, C101.1, C111.1, C112.1, C113.1, C114.1, C115.1, C116.1, C117.1, C8.1, C9.1, IC1.5 (VDDIO), IC1.8 (VDD), TP102.1, U1.1 (IOVDD), U1.10 (IOVDD), U1.22 (IOVDD), U1.33 (IOVDD), U1.42 (IOVDD), U1.43 (ADC_AVDD), U1.44 (VREG_IN), U1.48 (USB_VDD), U1.49 (IOVDD)
- net +3V3: now also J102.4; no longer J102.3
- net +5V: now also TP103.1
- net GND: now also J102.5, U102.1 (SH); no longer J102.4, U102.13 (SH)
- net LED_HB: now also U1.14 (GPIO11); no longer U1.37 (GPIO25)
- net RUN: now also J102.3; no longer J102.5
- net SWCLK: now also J102.10; no longer J102.2
- net SWD: now also J102.9; no longer J102.1
- net GPIO16: now reaches U1.27 (GPIO16)
- net GPIO16: now also J102.1
- net GPIO17: now reaches U1.28 (GPIO17)
- net GPIO17: now also J102.2
- net GPIO19: now reaches U1.30 (GPIO19)
- net GPIO19: now also J102.8
- net GPIO20: now reaches U1.31 (GPIO20)
- net GPIO20: now also J102.7
- net GPIO21: now reaches U1.32 (GPIO21)
- net GPIO21: now also J102.6
- net UART1_RX: no longer names the net of U1.12 (GPIO9)
- net UART1_RX: no longer J102.9
- net UART1_TX: no longer names the net of U1.11 (GPIO8)
- net UART1_TX: no longer J102.10
- no-connect marks 10 -> 21
Other:
- note added: "5V0->3V3 LDO"
- note added: "Debug"
- note added: "Force USB boot"
- note added: "IMU"
- note added: "MISC"
- note added: "RP2040"
- note added: "USB-C"
- moved on the sheet: C10, C101, C102, C103, C104, C105, C106, C107, C108, C109, C110, C111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
